File: PCB Shield/Mega_2560 core mini_full_2.0_PM/Mega_2560 core mini_full_2.0.sch (KiCad schematic (older format))
At the start: 107 parts, among them P1 2560-core, P10 SPI_libre, P11 Trim, P12 Stick_left, P13 Stick_right, P14 Switch, P15 LCD_I2C, P16 LCD, P17 Battery LIPO, P18 Ecolage, P19 Module_TX, P2 Clock, P20 Module_RS232/TTL, P21 Sw_power, P22 CONN_JQ6500_28P_mini, P23 Rot_1, P24 Rot_2, P25 Key_select_menu_ESC, P26 LCD_Vcc_select, P27 HP, P28 5v/3,3v manches, P3 Option, P4 Potentiometre, P5 Vibreur, P6 Micro_sd, P7 Option, P8 Audio, P9 SPI, U1 4066, U2 TLP290, U3 TLP290, U4 L4941, U5 LD1117S33TR, U6 MCP604-I/SL

Commit message: Update _Mega_2560 core mini_full_2.0_PM
Parts:
- removed P12: Stick_left, Pin_Headers:Pin_Header_Straight_1x04_Pitch2.54mm, symbol CONN_01X04
- removed P13: Stick_right, Pin_Headers:Pin_Header_Straight_1x04_Pitch2.54mm, symbol CONN_01X04
- removed P7: Option, Pin_Headers:Pin_Header_Straight_1x06_Pitch2.54mm, symbol CONN_01X06
- removed P8: Audio, Pin_Headers:Pin_Header_Straight_1x05_Pitch2.54mm, symbol CONN_01X05
- added C12, C13, C14: 100nF, Capacitors_SMD:C_1206, symbol C-RESCUE-Mega_2560_core_mini_full_2.0
- added P12: Stick_left, Pin_Headers:Pin_Header_Straight_2x03_Pitch2.54mm, symbol CONN_01X06
- added P13: Stick_right, Pin_Headers:Pin_Header_Straight_1x06_Pitch2.54mm, symbol CONN_01X06
- added P29: RXTX, Pin_Headers:Pin_Header_Straight_1x04_Pitch2.54mm, symbol CONN_01X04
- added P30: MiniDCDC3A, MiniDCDC3A, symbol CONN_01X08
- added P7: HF_modules, Pin_Headers:Pin_Header_Straight_1x09_Pitch2.54mm, symbol CONN_01X09
- added P8: Audio, Pin_Headers:Pin_Header_Straight_1x04_Pitch2.54mm, symbol CONN_01X04
- P17: value Battery LIPO -> BATT
- P20: value Module_RS232/TTL -> TTL/RS232
- P25: value Key_select_menu_ESC -> Keys
- P26: value LCD_Vcc_select -> LCD_Alim
- P4: value Potentiometre -> 3 Pots; footprint Pin_Headers:Pin_Header_Straight_2x05_Pitch2.54mm -> Pin_Headers:Pin_Header_Straight_3x03_Pitch2.54mm
Connections:
- net labels added: CS_CC2500, CS_CYRF6936, DCDC_IN+, LIPO+, R16_R17
- wire segments 431 -> 478
- no-connect marks 28 -> 23
Other:
- note added: "DCDC_IN-"
- note added: "Option module DCDC 3A"
- note removed: "+"
- note removed: "-"
- moved on the sheet: C11, C16, C17, C38, C5, C8, C9, D1, D2, P21, P5, R1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

Commit message: Update_Mega_2560 core mini_full_2.0_PM_23-8-2017
Parts:
- removed P4: 3 Pots, Pin_Headers:Pin_Header_Straight_3x03_Pitch2.54mm, symbol CONN_01X09
- removed P7: HF_modules, Pin_Headers:Pin_Header_Straight_1x09_Pitch2.54mm, symbol CONN_01X09
- removed U1: 4066, Librairie master:SOP14, symbol 4066
- added BT1: CR2032, Pin_Headers:Pin_Header_Straight_1x02_Pitch2.54mm, symbol BATTERY
- added C15, C18, C19, C20, C21, C22, C23: 100nF, Capacitors_SMD:C_1206, symbol C-RESCUE-Mega_2560_core_mini_full_2.0
- added D3, D4: LL4148, D_SCD80_HandSoldering, symbol DIODE
- added P31: Pot2, Pin_Headers:Pin_Header_Straight_1x03_Pitch2.54mm, symbol CONN_01X03
- added P32: Pot1, Pin_Headers:Pin_Header_Straight_1x03_Pitch2.54mm, symbol CONN_01X03
- added P4: Pot3, Pin_Headers:Pin_Header_Straight_1x03_Pitch2.54mm, symbol CONN_01X03
- added P7: SPIX, Pin_Header_Straight_2x05_Pitch2.54mm, symbol CONN_01X10
- added R10: 22K, Resistors_SMD:R_1206, symbol R-RESCUE-Mega_2560_core_mini_full_2.0
- added R15, R20: 10K, Resistors_SMD:R_1206, symbol R-RESCUE-Mega_2560_core_mini_full_2.0
- added U1: 74LVC1G3157, SOT-363_SC-70-6_Handsoldering, symbol 74LVC1G3157
- added U7: FM24W256, SOIC-8-FRAM_DI, symbol 24C512
- added U8: DS3231, SO-16-DS3231, symbol DS3231
- added U9: 4050, SO-16-N, symbol 4050-RESCUE-Mega_2560_core_mini_full_2.0
- R2: value 22K -> 1K
Connections:
- net labels added: CS_A7105, CS_NRF24L01, Hold_Power, JQ6500Busy, JQ6500Data, Master_PPMout, PPM16_SIMout, SCL, SDA, Sim_Control, Xmitter_MISO, Xmitter_MOSI, Xmitter_SCK
- net labels removed: PH2, PPM_out, R16_R17, RXD2, TXD2, core_pw10, core_pw13
- wire segments 478 -> 524
- no-connect marks 23 -> 15
Other:
- note added: "( Option si utilisation de la télémètrie )"
- note added: "(Module Interne\nMulti Protocoles)"
- note added: "Buzzer"
- note added: "Clock"
- note added: "Coupure Alim \n"
- note added: "Fram"
- note added: "Module HF"
- note removed: "Alim module"
- note removed: "Option si utilisation de la télémètrie"
- moved on the sheet: C1, C10, C12, C13, C14, C2, C28, C3, C31, C38, C5, C6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

Commit message: Update schematic R values
Parts:
- removed BT1: CR2032, Pin_Headers:Pin_Header_Straight_1x02_Pitch2.54mm, symbol BATTERY
- removed C1, C2, C3, C5: 47nF, Capacitors_SMD:C_1206, symbol C-RESCUE-Mega_2560_core_mini_full_2.0
- removed C10, C11, C12, C13, C14, C15, C16, C17, C18, C19, C20, C21, C22, C23, C26, C27, C29, C31, C32, C33, C34, C38, C4, C6, C9: 100nF, Capacitors_SMD:C_1206, symbol C-RESCUE-Mega_2560_core_mini_full_2.0
- removed C28, C7, C8: 47µF, Capacitors_SMD:CP_Elec_6.3x5.3, symbol CP1-RESCUE-Mega_2560_core_mini_full_2.0
- removed C42: 6.8nF, Capacitors_SMD:C_1206, symbol C-RESCUE-Mega_2560_core_mini_full_2.0
- removed C43, C44, C45, C46: 22nF, Capacitors_SMD:C_1206, symbol C-RESCUE-Mega_2560_core_mini_full_2.0
- removed D1, D2, D6: MBR0520, Diodes_SMD:D_SOD-123, symbol MBR0520
- removed D3, D4: LL4148, D_SCD80_HandSoldering, symbol DIODE
- removed P1: 2560-core, anthoperso:Connectors-2560-core, symbol 2560-core
- removed P10: SPI_libre, Pin_Headers:Pin_Header_Straight_1x03_Pitch2.54mm, symbol CONN_01X03
- removed P11: Trim, Pin_Headers:Pin_Header_Straight_2x05_Pitch2.54mm, symbol CONN_01X10
- removed P12: Stick_left, Pin_Headers:Pin_Header_Straight_2x03_Pitch2.54mm, symbol CONN_01X06
- removed P13: Stick_right, Pin_Headers:Pin_Header_Straight_1x06_Pitch2.54mm, symbol CONN_01X06
- removed P14: Switch, Pin_Headers:Pin_Header_Straight_2x05_Pitch2.54mm, symbol CONN_01X10
- removed P15: LCD_I2C, Pin_Headers:Pin_Header_Straight_1x04_Pitch2.54mm, symbol CONN_01X04
- removed P16: LCD, anthoperso:Pin_Header_Straight_2x10_Pitch2.54mm, symbol CONN_01X20
- removed P17: BATT, Pin_Headers:Pin_Header_Straight_1x02_Pitch2.54mm, symbol CONN_01X02
- removed P18: Ecolage, Pin_Headers:Pin_Header_Straight_1x02_Pitch2.54mm, symbol CONN_01X02
- removed P19: Module_TX, Pin_Headers:Pin_Header_Straight_2x04_Pitch2.54mm, symbol CONN_01X08
- removed P2: Clock, Pin_Headers:Pin_Header_Straight_1x04_Pitch2.54mm, symbol CONN_01X04
- removed P20: TTL/RS232, anthoperso:Con_RS232_TTL, symbol CONN_01X08
- removed P21: Sw_power, Pin_Headers:Pin_Header_Straight_1x02_Pitch2.54mm, symbol CONN_01X02
- removed P22: CONN_JQ6500_28P_mini, anthoperso:connector_mini-JQ6500-28P, symbol CONN_JQ6500_28P_mini-RESCUE-Mega_2560_core_mini_full_2.0
- removed P23: Rot_1, Pin_Headers:Pin_Header_Straight_1x04_Pitch2.54mm, symbol CONN_01X04
- removed P24: Rot_2, Pin_Headers:Pin_Header_Straight_1x04_Pitch2.54mm, symbol CONN_01X04
- removed P25: Keys, Pin_Headers:Pin_Header_Straight_2x04_Pitch2.54mm, symbol CONN_01X08
- removed P26: LCD_Alim, Pin_Headers:Pin_Header_Straight_1x03_Pitch2.54mm, symbol CONN_01X03
- removed P27: HP, Pin_Headers:Pin_Header_Straight_1x02_Pitch2.54mm, symbol CONN_01X02
- removed P28: 5v/3,3v manches, Pin_Headers:Pin_Header_Straight_1x03_Pitch2.54mm, symbol CONN_01X03
- removed P29: RXTX, Pin_Headers:Pin_Header_Straight_1x04_Pitch2.54mm, symbol CONN_01X04
- removed P3: Option, Pin_Headers:Pin_Header_Straight_1x04_Pitch2.54mm, symbol CONN_01X04
- removed P30: MiniDCDC3A, MiniDCDC3A, symbol CONN_01X08
- removed P31: Pot2, Pin_Headers:Pin_Header_Straight_1x03_Pitch2.54mm, symbol CONN_01X03
- removed P32: Pot1, Pin_Headers:Pin_Header_Straight_1x03_Pitch2.54mm, symbol CONN_01X03
- removed P4: Pot3, Pin_Headers:Pin_Header_Straight_1x03_Pitch2.54mm, symbol CONN_01X03
- removed P5: Vibreur, Pin_Headers:Pin_Header_Straight_1x02_Pitch2.54mm, symbol CONN_01X02
- removed P6: Micro_sd, Pin_Headers:Pin_Header_Straight_1x06_Pitch2.54mm, symbol CONN_01X06
- removed P7: SPIX, Pin_Header_Straight_2x05_Pitch2.54mm, symbol CONN_01X10
- removed P8: Audio, Pin_Headers:Pin_Header_Straight_1x04_Pitch2.54mm, symbol CONN_01X04
- removed P9: SPI, Pin_Headers:Pin_Header_Straight_2x03_Pitch2.54mm, symbol CONN_02X03
- removed R1, R10: 22K, Resistors_SMD:R_1206, symbol R-RESCUE-Mega_2560_core_mini_full_2.0
- removed R11, R12, R13, R14: 15K, Resistors_SMD:R_1206, symbol R-RESCUE-Mega_2560_core_mini_full_2.0
- removed R15, R20, R26, R28, R29, R31, R32, R34, R35, R37, R5, R6: 10K, Resistors_SMD:R_1206, symbol R-RESCUE-Mega_2560_core_mini_full_2.0
- removed R16: 2.7K, Resistors_SMD:R_1206, symbol R-RESCUE-Mega_2560_core_mini_full_2.0
- removed R17: 5.1K, Resistors_SMD:R_1206, symbol R-RESCUE-Mega_2560_core_mini_full_2.0
- removed R18, R19, R22, R23: 5.1k, Resistors_SMD:R_1206, symbol R-RESCUE-Mega_2560_core_mini_full_2.0
- removed R2, R4: 1K, Resistors_SMD:R_1206, symbol R-RESCUE-Mega_2560_core_mini_full_2.0
- removed R24, R25: 33K, Resistors_SMD:R_1206, symbol R-RESCUE-Mega_2560_core_mini_full_2.0
- removed R27, R30, R33, R36: POT_22k, Potentiometers:Potentiometer_Trimmer_Bourns_3296W, symbol POT-RESCUE-Mega_2560_core_mini_full_2.0
- removed R3: 18K, Resistors_SMD:R_1206, symbol R-RESCUE-Mega_2560_core_mini_full_2.0
- removed R7: 470, Resistors_SMD:R_1206, symbol R-RESCUE-Mega_2560_core_mini_full_2.0
- removed R8: 200, Resistors_SMD:R_1206, symbol R-RESCUE-Mega_2560_core_mini_full_2.0
- removed R9: 220, anthoperso:R_1206, symbol R-RESCUE-Mega_2560_core_mini_full_2.0
- removed RV1: 220K, Potentiometers:Potentiometer_Trimmer_Bourns_3296W, symbol POT-RESCUE-Mega_2560_core_mini_full_2.0
- removed RV2, RV3, RV4, RV5: POT_100k, Potentiometers:Potentiometer_Bourns_3296W_3-8Zoll_Inline_ScrewUp, symbol POT-RESCUE-Mega_2560_core_mini_full_2.0
- removed RV6: 22K, Potentiometers:Potentiometer_Trimmer_Bourns_3296W, symbol POT-RESCUE-Mega_2560_core_mini_full_2.0
- removed U1: 74LVC1G3157, SOT-363_SC-70-6_Handsoldering, symbol 74LVC1G3157
- removed U2, U3: TLP290, anthoperso:SOP4, symbol TLP290-RESCUE-Mega_2560_core_mini_full_2.0
- removed U4: L4941, Power_Integrations:TO-220, symbol L4941
- removed U5: LD1117S33TR, TO_SOT_Packages_SMD:SOT-223, symbol LD1117S33TR
- removed U6: MCP604-I/SL, Librairie master:SOP14, symbol MCP6004
- removed U7: FM24W256, SOIC-8-FRAM_DI, symbol 24C512
- removed U8: DS3231, SO-16-DS3231, symbol DS3231
- removed U9: 4050, SO-16-N, symbol 4050-RESCUE-Mega_2560_core_mini_full_2.0
- removed W1, W2, W3, W4: TEST_2P, anthoperso:TESTPT, symbol TEST_2P
Connections:
- no-connect marks 15 -> 0
Other:
- note removed: "( Option si utilisation de la télémètrie )"
- note removed: "(Module Interne\nMulti Protocoles)"
- note removed: "+3.3V\n"
- note removed: "+5V"
- note removed: "Buzzer"
- note removed: "Clock"
- note removed: "Coupure Alim \n"
- note removed: "DCDC_IN-"
- note removed: "Fram"
- note removed: "Isolation Module TTL"
- note removed: "Module HF"
- note removed: "Option Amplification des sticks (Fonctionne sans)"
- note removed: "Option module DCDC 3A"
- note removed: "Option si utilisation du 3.3V dans le montage"
- note removed: "PPM Management"
- note removed: "Power Management"
- note removed: "Power Switch"
- note removed: "Stick control"
